File: Keyboard_Tutorial.sch (KiCad schematic (older format))
At the start: 24 parts, among them SW1 SW_Push, U1 ATmega32U4-AU, Y1 16MHz

Commit message: Add submodules
Parts:
- removed Y1: 16MHz, Crystal:Crystal_SMD_3225-4Pin_3.2x2.5mm, symbol Device:Crystal_GND23_Small
- added Y?: Crystal_GND24_Small, symbol Device:Crystal_GND24_Small
- renumbered MX3 to MX2, MX2 to MX3
Connections:
- net GND: now also Y?.2, Y?.4
- net at C2.1, U1.16 (XTAL2): now also Y?.3
- net at C1.2, U1.17 (XTAL1): now also Y?.1
Changed lines of the file:
@@
 	2800 1950 2800 2250
-$Comp
-L Device:Crystal_GND23_Small Y1
-U 1 1 6478B987
-P 3250 2150
-F 0 "Y1" H 3394 2196 50  0000 L CNN
-F 1 "16MHz" H 3394 2105 50  0000 L CNN
-F 2 "Crystal:Crystal_SMD_3225-4Pin_3.2x2.5mm" H 3250 2150 50  0001 C CNN
-F 3 "~" H 3250 2150 50  0001 C CNN
-	1    3250 2150
-	1    0    0    -1
-$EndComp
-Connection ~ 3250 2050
 $Comp
 L Device:C_Small C2
@@
 	2800 2250 2900 2250
 Wire Wire Line
-	3100 2250 3250 2250
-Wire Wire Line
-	4000 2250 3250 2250
-Connection ~ 3250 2250
-Wire Wire Line
 	3350 2150 3350 2350
 Wire Wire Line
@@
 $EndComp
 $Comp
-L MX_Alps_Hybrid:MX-NoLED MX2
+L MX_Alps_Hybrid:MX-NoLED MX3
 U 1 1 648030F7
 P 7550 2500
-F 0 "MX2" H 7583 2723 60  0000 C CNN
+F 0 "MX3" H 7583 2723 60  0000 C CNN
 F 1 "MX-NoLED" H 7583 2649 20  0000 C CNN
 F 2 "MX_Alps_Hybrid:MX-1U" H 6925 2475 60  0001 C CNN
@@
 $EndComp
 $Comp
-L MX_Alps_Hybrid:MX-NoLED MX3
+L MX_Alps_Hybrid:MX-NoLED MX2
 U 1 1 648035D5
 P 6900 3100
-F 0 "MX3" H 6933 3323 60  0000 C CNN
+F 0 "MX2" H 6933 3323 60  0000 C CNN
 F 1 "MX-NoLED" H 6933 3249 20  0000 C CNN
 F 2 "MX_Alps_Hybrid:MX-1U" H 6275 3075 60  0001 C CNN
@@
 Wire Wire Line
 	3550 3400 3550 3450
+Wire Wire Line
+	3100 2250 3250 2250
+$Comp
+L Device:Crystal_GND24_Small Y?
+U 1 1 64786AFA
+P 3250 2150
+F 0 "Y?" V 3204 2294 50  0000 L CNN
+F 1 "Crystal_GND24_Small" V 3295 2294 50  0000 L CNN
+F 2 "" H 3250 2150 50  0001 C CNN
+F 3 "~" H 3250 2150 50  0001 C CNN
+	1    3250 2150
+	0    1    1    0
+$EndComp
+Connection ~ 3250 2050
+Connection ~ 3250 2250
+Wire Wire Line
+	3250 2250 4000 2250
 $EndSCHEMATC

Commit message: Add submodules
Parts:
- Y1: renamed from Y?; footprint (none) -> Crystal:Crystal_SMD_3225-4Pin_3.2x2.5mm
Changed lines of the file:
@@
 	3100 2250 3250 2250
 $Comp
-L Device:Crystal_GND24_Small Y?
+L Device:Crystal_GND24_Small Y1
 U 1 1 64786AFA
 P 3250 2150
-F 0 "Y?" V 3204 2294 50  0000 L CNN
+F 0 "Y1" V 3204 2294 50  0000 L CNN
 F 1 "Crystal_GND24_Small" V 3295 2294 50  0000 L CNN
-F 2 "" H 3250 2150 50  0001 C CNN
+F 2 "Crystal:Crystal_SMD_3225-4Pin_3.2x2.5mm" H 3250 2150 50  0001 C CNN
 F 3 "~" H 3250 2150 50  0001 C CNN
 	1    3250 2150
